Commit message: fix transformation error from transform component

File: robotname_description/urdf/robotname.urdf (robot description, URDF)
Before this commit: robot sam_bot, 7 links, 6 joints
Links:
- removed link camera_depth_frame
Joints:
- removed joint camera_depth_joint

Commit message: rtabmap slam branch

File: robotname_description/urdf/robotname.urdf (robot description, URDF)
Before this commit: robot sam_bot, 6 links, 5 joints
Links:
- added link camera_optical_link
Joints:
- added joint camera_joint_optic: type fixed, parent camera_link, child camera_optical_link, origin xyz=0.215 0 0.05 rpy=${-pi/2} 0 ${-pi/2}
