Commit message: nav2 omni pure pursuit  heading error

File: robotname_description/urdf/robotomni.urdf (robot description, URDF)
Before this commit: robot robotomni, 3 links, 2 joints
Links:
- added link lidar_link, mass 0.125; collision cylinder length=0.055 radius=0.0508; visual cylinder length=0.055 radius=0.0508
Joints:
- added joint lidar_joint: type fixed, parent base_link, child lidar_link, origin xyz=0.35 0 0.04 rpy=0 0 0
- joint base_joint: child base_footprint -> base_link; parent base_link -> base_footprint
