Commit message: add alot of behavior and use yolo for obj detection

File: robotname_description/urdf/realomni.urdf (robot description, URDF)
Before this commit: robot realomni, 4 links, 3 joints
Joints:
- joint base_joint: child base_link -> base_footprint; parent base_footprint -> base_link
- joint lidar_joint: origin xyz=-0.30 0.10 0 rpy=3.14 0 2.6172 -> xyz=-0.40 0.20 0 rpy=0 0 2.0944
- joint odom_joint: child base_odom -> base_link; origin xyz=-0.25 0 0 -> xyz=0.28 0 0; parent base_link -> base_odom

Commit message: migrasi ke pc baru

File: robotname_description/urdf/realomni.urdf (robot description, URDF)
Before this commit: robot realomni, 4 links, 3 joints
Links:
- added link omnicam_link
Joints:
- added joint ocam_joint: type fixed, parent base_link, child omnicam_link, origin xyz=0.150 0 0
- joint lidar_joint: origin xyz=-0.40 0.20 0 rpy=0 0 2.0944 -> xyz=-0.272 0.19 0 rpy=3.14 0 2.0944
- joint odom_joint: origin xyz=0.28 0 0 -> xyz=0.3 0 0

Commit message: alot of changes

File: robotname_description/urdf/realomni.urdf (robot description, URDF)
Before this commit: robot realomni, 5 links, 4 joints
Joints:
- joint ocam_joint: origin xyz=0.150 0 0 -> xyz=0.170 0 0

Commit message: update 19 mei

File: robotname_description/urdf/realomni.urdf (robot description, URDF)
Before this commit: robot realomni, 5 links, 4 joints
Links:
- added link camera_link
Joints:
- added joint camera_joint: type fixed, parent base_link, child camera_link, origin xyz=0.32 0.0 0.692 rpy=0.0 0.523599 0.0
- joint lidar_joint: origin xyz=-0.272 0.19 0 rpy=3.14 0 2.0944 -> xyz=-0.220 0.210 0 rpy=3.14 0 2.0944

Commit message: move lidar package to urg node 2, add move  with lidar reference plugins

File: robotname_description/urdf/realomni.urdf (robot description, URDF)
Before this commit: robot realomni, 6 links, 5 joints
Joints:
- joint camera_joint: origin xyz=0.32 0.0 0.692 rpy=0.0 0.523599 0.0 -> xyz=0.32 0.0 0.692 rpy=0.0 0.349066 0.0

Commit message: muavang

File: robotname_description/urdf/realomni.urdf (robot description, URDF)
Before this commit: robot realomni, 6 links, 5 joints
Joints:
- joint camera_joint: origin xyz=0.32 0.0 0.692 rpy=0.0 0.349066 0.0 -> xyz=0.15 0.0 0.692 rpy=0.0 0.261799 0.0

Commit message: bisa camera silo

File: robotname_description/urdf/realomni.urdf (robot description, URDF)
Before this commit: robot realomni, 6 links, 5 joints
Joints:
- joint lidar_joint: origin xyz=-0.220 0.210 0 rpy=3.14 0 2.0944 -> xyz=-0.25 -0.195 0 rpy=3.14 0 -2.09

Commit message: perubahan akhir

File: robotname_description/urdf/realomni.urdf (robot description, URDF)
Before this commit: robot realomni, 6 links, 5 joints
Links:
- removed link camera_link
- added link camera1_link
Joints:
- joint camera_joint: child camera_link -> camera1_link

Commit message: add robot new urdf

File: robotname_description/urdf/realomni.urdf (robot description, URDF)
Before this commit: robot realomni, 6 links, 5 joints
Links:
- added link camera2_link
- added link laser2
Joints:
- added joint camera2_joint: type fixed, parent base_link, child camera2_link, origin xyz=-0.15 0.0 0.2 rpy=0.0 0.0 0.0
- added joint lidar_joint2: type fixed, parent base_link, child laser2, origin xyz=-0.25 0.195 0 rpy=3.14 0 2.09

Commit message: merger 2 data lidar dengan iratools

File: robotname_description/urdf/realomni.urdf (robot description, URDF)
Before this commit: robot realomni, 8 links, 7 joints
Joints:
- joint camera2_joint: origin xyz=-0.15 0.0 0.2 rpy=0.0 0.0 0.0 -> xyz=-0.32 0.0 0.22 rpy=0.0 0.0 0.0

Commit message: detection camera sudah bisa

File: robotname_description/urdf/realomni.urdf (robot description, URDF)
Before this commit: robot realomni, 8 links, 7 joints
Joints:
- joint camera2_joint: origin xyz=-0.32 0.0 0.22 rpy=0.0 0.0 0.0 -> xyz=-0.32 0.0 0.22 rpy=0.0 0.0 -3.14
